File: H_bridge.kicad_sch (KiCad schematic)
At the start: 17 parts, among them J801 track out, J802 track out, U801 L298N

Commit message: added hierarchial labels to some schematics
Parts:
- renumbered C802 to C4, C804 to C5, C801 to C6, C803 to C7, D806 to D10, D808 to D11, D801 to D4, D803 to D5, D805 to D6, D807 to D7, D802 to D8, D804 to D9, J801 to J8, J802 to J9, R801 to R22, R802 to R23, U801 to U7

Commit message: moved some schematic scheets to their own folders and routed a board with it. This allow for re-use of PCB parts.
Parts:
- renumbered C6 to C801, C4 to C802, C7 to C803, C5 to C804, D4 to D801, D8 to D802, D5 to D803, D9 to D804, D6 to D805, D10 to D806, D7 to D807, D11 to D808, J8 to J801, J9 to J802, R22 to R801, R23 to R802, U7 to U801
