File: EEPROM/EEPROM.kicad_sch (KiCad schematic)
At the start: 2 parts, among them U1901 24LC256

Commit message: removed hierarchial labels for power symbols and replaced them with actual power symbols also updated footprint of the inductor of the 5V buck
Parts:
- renumbered C1901 to C801, U1901 to U801
Changed lines of the file:
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@@
 (kicad_sch (version 20230121) (generator eeschema)
   (paper "A4")
-  (junction (at 118.11 100.33) (diameter 0) (color 0 0 0 0)
-  )
   (junction (at 107.95 76.2) (diameter 0) (color 0 0 0 0)
   )
@@
     (stroke (width 0) (type default))
   )
-  (wire (pts (xy 118.11 100.33) (xy 119.38 100.33))
-    (stroke (width 0) (type default))
-  )
   (wire (pts (xy 96.52 88.9) (xy 97.79 88.9))
     (stroke (width 0) (type default))
@@
     (effects (font (size 1.27 1.27)) (justify left))
   )
-  (hierarchical_label "GND" (shape passive) (at 119.38 100.33 0) (fields_autoplaced)
-    (effects (font (size 1.27 1.27)) (justify left))
-  )
   (hierarchical_label "A2" (shape passive) (at 96.52 88.9 180) (fields_autoplaced)
     (effects (font (size 1.27 1.27)) (justify right))
@@
   (symbol (lib_id "power:+5V") (at 107.95 72.39 0) (unit 1)
     (in_bom yes) (on_board yes) (dnp no) (fields_autoplaced)
-    (property "Reference" "#PWR0154" (at 107.95 76.2 0)
+    (property "Reference" "#PWR0801" (at 107.95 76.2 0)
       (effects (font (size 1.27 1.27)) hide)
     )
@@
   (symbol (lib_id "Memory_EEPROM:24LC256") (at 107.95 86.36 0) (unit 1)
     (in_bom yes) (on_board yes) (dnp no) (fields_autoplaced)
-    (property "Reference" "U1901" (at 109.9694 77.5802 0)
+    (property "Reference" "U801" (at 109.9694 77.5802 0)
       (effects (font (size 1.27 1.27)) (justify left))
     )
@@
     )
   )
+  (symbol (lib_id "power:GND") (at 107.95 100.33 0) (unit 1)
+    (in_bom yes) (on_board yes) (dnp no) (fields_autoplaced)
+    (property "Reference" "#PWR0802" (at 107.95 106.68 0)
+      (effects (font (size 1.27 1.27)) hide)
+    )
+    (property "Value" "GND" (at 107.95 105.41 0)
+      (effects (font (size 1.27 1.27)))
+    )
+    (property "Footprint" "" (at 107.95 100.33 0)
+      (effects (font (size 1.27 1.27)) hide)
+    )
+    (property "Datasheet" "" (at 107.95 100.33 0)
+      (effects (font (size 1.27 1.27)) hide)
+    )
+    (pin "1")
+    (instances
+      (project "EEPROM"
+        (path "/7726f3b0-6d28-4a62-ae77-022bfbf3ad3f"
+          (reference "#PWR0802") (unit 1)
+        )
+      )
+    )
+  )
   (symbol (lib_id "Device:C") (at 85.09 83.82 0) (mirror x) (unit 1)
     (in_bom yes) (on_board yes) (dnp no) (fields_autoplaced)
-    (property "Reference" "C1901" (at 82.169 82.9853 0)
+    (property "Reference" "C801" (at 82.169 82.9853 0)
       (effects (font (size 1.27 1.27)) (justify right))
     )
